File: NDriveShield.kicad_pcb (KiCad board)
At the start: 2 copper layers, 68.6 x 53.3 mm, 23 parts, among them Q1 NTD5867NLT4G, Q2 NTD5867NLT4G, Q3 NTD5867NLT4G, Q4 NTD5867NLT4G, Q5 NTD5867NLT4G, Q6 NTD5867NLT4G, SW1 SW_PUSHBUTTON

Commit message: #4 Make compatible to KiCAD nightly
Signed-off-by: Tisham Dhar <whatnickd@gmail.com>
Other:
- outline, holes or cut-outs redrawn
- net class Default removed
- net class Power removed
